Commit message: Step 1: buoyancy + hydrodynamic drag — AUV hovers at z=1.2

File: src/srmauv_description/urdf/srmauv.urdf.xacro (robot description, xacro)
@@ -18,12 +18,4 @@
   <xacro:property name="cy" value="-0.156"/>
   <xacro:property name="cz" value="-0.117"/>
-  <!-- Massless root link: robot_state_publisher/KDL rejects a root link that
-       carries inertia, so base_link hangs off this dummy via a fixed joint. -->
-  <link name="base_footprint"/>
-  <joint name="base_joint" type="fixed">
-    <parent link="base_footprint"/>
-    <child link="base_link"/>
-    <origin xyz="0 0 0" rpy="0 0 0"/>
-  </joint>
   <link name="base_link">
     <!-- Full detail mesh for appearance. -->
@@ -56,3 +48,28 @@
   <!-- No <material> override here on purpose: that would replace the COLLADA
        per-part colors with a flat color. The .dae carries its own materials. -->
+  <!-- ================================================================
+       STEP 1: Underwater Dynamics
+       Buoyancy: volume=0.020 m^3 = mass(20kg)/water_density(1000)
+                 -> exact neutral buoyancy as the baseline.
+                 With drag now present, this won't fly away.
+       Drag: cd_linear=10, cd_quadratic=50 N/(m/s)^2, cd_angular=5
+             These are realistic starting values for a 0.6m AUV.
+       ================================================================ -->
+  <gazebo>
+    <plugin name="buoyancy_plugin" filename="libBuoyancyPlugin.so">
+      <fluid_density>1000</fluid_density>
+      <link name="base_link">
+        <center_of_volume>0.0 -0.156 -0.117</center_of_volume>
+        <volume>0.020</volume>
+      </link>
+    </plugin>
+  </gazebo>
+  <gazebo>
+    <plugin name="hydrodynamic_plugin" filename="libhydrodynamic_plugin.so">
+      <cd_linear>10.0</cd_linear>
+      <cd_quadratic>50.0</cd_quadratic>
+      <cd_angular>5.0</cd_angular>
+      <fluid_level>2.5</fluid_level>
+    </plugin>
+  </gazebo>
 </robot>

Commit message: Step 2: fix thruster yaw/strafe mixing, tune drag damping, bake plugin path into launch file

File: src/srmauv_description/urdf/srmauv.urdf.xacro (robot description, xacro)
@@ -1,23 +1,14 @@
 <?xml version="1.0"?>
 <robot name="srmauv" xmlns:xacro="http://www.ros.org/wiki/xacro">
-  <!-- ============================================================
-       Geometry derived from "AUV Vehicle full assembly v4.step":
-         bounding box ~ 0.587 x 0.601 x 0.435 m
-         center offset ~ (0, -0.156, -0.117) m from the STEP origin
-       STL is in millimetres -> Gazebo metres, so mesh_scale = 0.001.
-       ============================================================ -->
   <xacro:property name="mesh_scale" value="0.001 0.001 0.001"/>
-  <xacro:property name="mesh_rpy"   value="0 0 0"/>
-  <xacro:property name="mass"       value="20.0"/>   <!-- kg, approx -->
-  <!-- Bounding-box dimensions (m) used for the simplified collision. -->
+  <xacro:property name="mesh_rpy"   value="0 0 1.5708"/>
+  <xacro:property name="mass"       value="20.0"/>
   <xacro:property name="bx" value="0.587"/>
   <xacro:property name="by" value="0.601"/>
   <xacro:property name="bz" value="0.435"/>
-  <!-- Center of the bounding box, relative to the STEP origin (m). -->
   <xacro:property name="cx" value="0.0"/>
   <xacro:property name="cy" value="-0.156"/>
-  <xacro:property name="cz" value="-0.117"/>
+  <xacro:property name="cz" value="-0.25"/>
   <link name="base_link">
-    <!-- Full detail mesh for appearance. -->
     <visual>
       <origin xyz="0 0 0" rpy="${mesh_rpy}"/>
@@ -27,6 +18,4 @@
       </geometry>
     </visual>
-    <!-- Simple box collision: a 1M-facet mesh collision would cripple
-         physics. Swap to a closer hull later if you need fine contacts. -->
     <collision>
       <origin xyz="${cx} ${cy} ${cz}" rpy="0 0 0"/>
@@ -38,6 +27,4 @@
       <origin xyz="${cx} ${cy} ${cz}" rpy="0 0 0"/>
       <mass value="${mass}"/>
-      <!-- Solid-box inertia for the bounding box (ixx etc. computed
-           from bx,by,bz and mass). Replace with CAD inertia if needed. -->
       <inertia
         ixx="${(1.0/12.0)*mass*(by*by + bz*bz)}" ixy="0.0" ixz="0.0"
@@ -46,14 +33,5 @@
     </inertial>
   </link>
-  <!-- No <material> override here on purpose: that would replace the COLLADA
-       per-part colors with a flat color. The .dae carries its own materials. -->
-  <!-- ================================================================
-       STEP 1: Underwater Dynamics
-       Buoyancy: volume=0.020 m^3 = mass(20kg)/water_density(1000)
-                 -> exact neutral buoyancy as the baseline.
-                 With drag now present, this won't fly away.
-       Drag: cd_linear=10, cd_quadratic=50 N/(m/s)^2, cd_angular=5
-             These are realistic starting values for a 0.6m AUV.
-       ================================================================ -->
+  <!-- STEP 1: Buoyancy -->
   <gazebo>
     <plugin name="buoyancy_plugin" filename="libBuoyancyPlugin.so">
@@ -65,11 +43,17 @@
     </plugin>
   </gazebo>
+  <!-- STEP 1: Hydrodynamic drag -->
   <gazebo>
     <plugin name="hydrodynamic_plugin" filename="libhydrodynamic_plugin.so">
-      <cd_linear>10.0</cd_linear>
+      <cd_linear>35.0</cd_linear>
       <cd_quadratic>50.0</cd_quadratic>
-      <cd_angular>5.0</cd_angular>
+      <cd_angular>25.0</cd_angular>
       <fluid_level>2.5</fluid_level>
     </plugin>
   </gazebo>
+  <!-- STEP 2: All 6 thrusters — single plugin on base_link -->
+  <gazebo>
+    <plugin name="all_thrusters_plugin" filename="libthruster_plugin.so">
+    </plugin>
+  </gazebo>
 </robot>

Commit message: Step 3: IMU, depth sensor, front and bottom cameras - all verified

File: src/srmauv_description/urdf/srmauv.urdf.xacro (robot description, xacro)
@@ -57,3 +57,125 @@
     </plugin>
   </gazebo>
+  <!-- ================================================================
+       STEP 3: Sensors
+       IMU, Depth, Front Camera, Bottom Camera
+       ================================================================ -->
+  <!-- IMU -->
+  <link name="imu_link"/>
+  <joint name="imu_joint" type="fixed">
+    <parent link="base_link"/>
+    <child link="imu_link"/>
+    <origin xyz="0 0 0" rpy="0 0 0"/>
+  </joint>
+  <gazebo reference="imu_link">
+    <sensor name="imu_sensor" type="imu">
+      <always_on>true</always_on>
+      <update_rate>100</update_rate>
+      <plugin name="imu_plugin" filename="libgazebo_ros_imu_sensor.so">
+        <ros>
+          <namespace>/srmauv</namespace>
+          <remapping>~/out:=imu</remapping>
+        </ros>
+        <initial_orientation_as_reference>false</initial_orientation_as_reference>
+      </plugin>
+    </sensor>
+  </gazebo>
+  <!-- Depth sensor (using altimeter as pressure proxy) -->
+  <link name="depth_link"/>
+  <joint name="depth_joint" type="fixed">
+    <parent link="base_link"/>
+    <child link="depth_link"/>
+    <origin xyz="0 0 -0.1" rpy="0 0 0"/>
+  </joint>
+  <gazebo reference="depth_link">
+    <sensor name="depth_sensor" type="ray">
+      <always_on>true</always_on>
+      <update_rate>50</update_rate>
+      <ray>
+        <scan>
+          <horizontal>
+            <samples>1</samples>
+            <resolution>1</resolution>
+            <min_angle>0</min_angle>
+            <max_angle>0</max_angle>
+          </horizontal>
+        </scan>
+        <range>
+          <min>0.01</min>
+          <max>10.0</max>
+          <resolution>0.001</resolution>
+        </range>
+      </ray>
+      <plugin name="depth_plugin" filename="libgazebo_ros_ray_sensor.so">
+        <ros>
+          <namespace>/srmauv</namespace>
+          <remapping>~/out:=depth</remapping>
+        </ros>
+        <output_type>sensor_msgs/Range</output_type>
+        <frame_name>depth_link</frame_name>
+      </plugin>
+    </sensor>
+  </gazebo>
+  <!-- Front camera -->
+  <link name="front_camera_link"/>
+  <joint name="front_camera_joint" type="fixed">
+    <parent link="base_link"/>
+    <child link="front_camera_link"/>
+    <origin xyz="0.29 0 0" rpy="0 0 0"/>
+  </joint>
+  <gazebo reference="front_camera_link">
+    <sensor name="front_camera" type="camera">
+      <always_on>true</always_on>
+      <update_rate>30</update_rate>
+      <camera>
+        <horizontal_fov>1.3962634</horizontal_fov>
+        <image>
+          <width>640</width>
+          <height>480</height>
+          <format>R8G8B8</format>
+        </image>
+        <clip><near>0.1</near><far>20</far></clip>
+      </camera>
+      <plugin name="front_camera_plugin" filename="libgazebo_ros_camera.so">
+        <ros>
+          <namespace>/srmauv</namespace>
+          <remapping>~/image_raw:=camera/front/image_raw</remapping>
+          <remapping>~/camera_info:=camera/front/camera_info</remapping>
+        </ros>
+        <camera_name>front_camera</camera_name>
+        <frame_name>front_camera_link</frame_name>
+      </plugin>
+    </sensor>
+  </gazebo>
+  <!-- Bottom camera -->
+  <link name="bottom_camera_link"/>
+  <joint name="bottom_camera_joint" type="fixed">
+    <parent link="base_link"/>
+    <child link="bottom_camera_link"/>
+    <origin xyz="0 0 -0.2" rpy="0 1.5708 0"/>
+  </joint>
+  <gazebo reference="bottom_camera_link">
+    <sensor name="bottom_camera" type="camera">
+      <always_on>true</always_on>
+      <update_rate>30</update_rate>
+      <camera>
+        <horizontal_fov>1.3962634</horizontal_fov>
+        <image>
+          <width>640</width>
+          <height>480</height>
+          <format>R8G8B8</format>
+        </image>
+        <clip><near>0.1</near><far>10</far></clip>
+      </camera>
+      <plugin name="bottom_camera_plugin" filename="libgazebo_ros_camera.so">
+        <ros>
+          <namespace>/srmauv</namespace>
+          <remapping>~/image_raw:=camera/bottom/image_raw</remapping>
+          <remapping>~/camera_info:=camera/bottom/camera_info</remapping>
+        </ros>
+        <camera_name>bottom_camera</camera_name>
+        <frame_name>bottom_camera_link</frame_name>
+      </plugin>
+    </sensor>
+  </gazebo>
 </robot>
